Commit message: - add gazebo launch file - add ros2 control - Advancement urdf (xacro)

File: description/robot.urdf.xacro (robot description, xacro)
@@ -2,228 +2,13 @@
 <robot xmlns:xacro="http://www.ros.org/wiki/xacro" name="ur5e">
     <link name="world" />
-    <joint name="joint_base" type="fixed">
-        <parent link="world" />
-        <child link="link_base" />
-        <origin xyz="0 0 0" rpy="0 0 0" />
-    </joint>
-    <link name="link_base">
-        <visual>
-            <origin xyz="0 0 0" rpy="0 0 ${pi}" />
-            <geometry>
-                <mesh filename="file://$(find ros2_robot_ur5e)/meshes/ur5e/visual/base.dae" />
-            </geometry>
-        </visual>
-        <collision>
-            <origin xyz="0 0 0" rpy="0 0 ${pi}" />
-            <geometry>
-                <mesh filename="file://$(find ros2_robot_ur5e)/meshes/ur5e/collision/base.stl" />
-            </geometry>
-        </collision>
-        <inertial>
-            <mass value="4.0" />
-            <origin rpy="0 0 0" xyz="0 0 0" />
-            <inertia
-                ixx="0.0044333156" ixy="0.0" ixz="0.0"
-                iyy="0.0044333156" iyz="0.0"
-                izz="0.0072" />
-        </inertial>
-    </link>
-    <joint name="joint_shoulder_pan" type="revolute">
-        <parent link="link_base" />
-        <child link="link_shoulder" />
-        <origin xyz="0 0 0.1625" rpy="0 0 0" />
-        <axis xyz="0 0 1" />
-        <limit lower="${-2*pi}" upper="${2*pi}" effort="150.0" velocity="${pi}" />
-        <dynamics damping="0" friction="0" />
-    </joint>
-    <link name="link_shoulder">
-        <visual>
-            <origin xyz="0 0 0" rpy="0 0 ${pi}" />
-            <geometry>
-                <mesh filename="file://$(find ros2_robot_ur5e)/meshes/ur5e/visual/shoulder.dae" />
-            </geometry>
-        </visual>
-        <collision>
-            <origin xyz="0 0 0" rpy="0 0 ${pi}" />
-            <geometry>
-                <mesh filename="file://$(find ros2_robot_ur5e)/meshes/ur5e/collision/shoulder.stl" />
-            </geometry>
-        </collision>
-        <inertial>
-            <mass value="3.761" />
-            <origin rpy="0.0 0.0 0.0" xyz="0.0 -0.00193 -0.02561" />
-            <inertia
-                ixx="0.0102675" ixy="0.0" ixz="0.0"
-                iyy="0.0102675" iyz="0.0"
-                izz="0.00666" />
-        </inertial>
-    </link>
-    <joint name="joint_shoulder_lift" type="revolute">
-        <parent link="link_shoulder" />
-        <child link="link_upper_arm" />
-        <origin xyz="0 0 0" rpy="${pi/2} 0 0" />
-        <axis xyz="0 0 1" />
-        <limit lower="${-2*pi}" upper="${2*pi}" effort="150.0" velocity="${pi}" />
-        <dynamics damping="0" friction="0" />
-    </joint>
-    <link name="link_upper_arm">
-        <visual>
-            <origin xyz="0 0 0.138" rpy="${pi/2} 0 ${-pi/2}" />
-            <geometry>
-                <mesh filename="file://$(find ros2_robot_ur5e)/meshes/ur5e/visual/upperarm.dae" />
-            </geometry>
-        </visual>
-        <collision>
-            <origin xyz="0 0 0.138" rpy="${pi/2} 0 ${-pi/2}" />
-            <geometry>
-                <mesh filename="file://$(find ros2_robot_ur5e)/meshes/ur5e/collision/upperarm.stl" />
-            </geometry>
-        </collision>
-        <inertial>
-            <mass value="8.058" />
-            <origin rpy="0.0 ${pi/2} 0.0" xyz="-0.2125 0.0 0.11336" />
-            <inertia
-                ixx="0.13388583542" ixy="0.0" ixz="0.0"
-                iyy="0.13388583542" iyz="0.0"
-                izz="0.0151074" />
-        </inertial>
-    </link>
-    <joint name="joint_elbow" type="revolute">
-        <parent link="link_upper_arm" />
-        <child link="link_forearm" />
-        <origin xyz="-0.425 0 0" rpy="0 0 0" />
-        <axis xyz="0 0 1" />
-        <limit lower="${-pi}" upper="${pi}" effort="150.0" velocity="${pi}" />
-        <dynamics damping="0" friction="0" />
-    </joint>
-    <link name="link_forearm">
-        <visual>
-            <origin xyz="0 0 0.007" rpy="${pi/2} 0 ${-pi/2}" />
-            <geometry>
-                <mesh filename="file://$(find ros2_robot_ur5e)/meshes/ur5e/visual/forearm.dae" />
-            </geometry>
-        </visual>
-        <collision>
-            <origin xyz="0 0 0.007" rpy="${pi/2} 0 ${-pi/2}" />
-            <geometry>
-                <mesh filename="file://$(find ros2_robot_ur5e)/meshes/ur5e/collision/forearm.stl" />
-            </geometry>
-        </collision>
-        <inertial>
-            <mass value="2.846" />
-            <origin rpy="0.0 ${pi/2} 0.0" xyz="-0.2422 0.0 0.0265" />
-            <inertia
-                ixx="0.03120936758" ixy="0.0" ixz="0.0"
-                iyy="0.03120936758" iyz="0.0"
-                izz="0.004095" />
-        </inertial>
-    </link>
-    <joint name="joint_wrist_1" type="revolute">
-        <parent link="link_forearm" />
-        <child link="link_wrist_1" />
-        <origin xyz="-0.3922 0 0.1333" rpy="0 0 0" />
-        <axis xyz="0 0 1" />
-        <limit lower="${-2*pi}" upper="${2*pi}" effort="28.0" velocity="${pi}" />
-        <dynamics damping="0" friction="0" />
-    </joint>
-    <link name="link_wrist_1">
-        <visual>
-            <origin xyz="0 0 -0.127" rpy="${pi/2} 0 0" />
-            <geometry>
-                <mesh filename="file://$(find ros2_robot_ur5e)/meshes/ur5e/visual/wrist1.dae" />
-            </geometry>
-        </visual>
-        <collision>
-            <origin xyz="0 0 -0.127" rpy="${pi/2} 0 0" />
-            <geometry>
-                <mesh filename="file://$(find ros2_robot_ur5e)/meshes/ur5e/collision/wrist1.stl" />
-            </geometry>
-        </collision>
-        <inertial>
-            <mass value="1.37" />
-            <origin rpy="0.0 0.0 0.0" xyz="0.0 -0.01634 -0.0018" />
-            <inertia
-                ixx="0.0025599" ixy="0.0" ixz="0.0"
-                iyy="0.0025599" iyz="0.0"
-                izz="0.0021942" />
-        </inertial>
-    </link>
-    <joint name="joint_wrist_2" type="revolute">
-        <parent link="link_wrist_1" />
-        <child link="link_wrist_2" />
-        <origin xyz="0 -0.0997 -2.044881182297852e-11" rpy="${pi/2} 0 0" />
-        <axis xyz="0 0 1" />
-        <limit lower="${-2*pi}" upper="${2*pi}" effort="${28.0}" velocity="${pi}" />
-        <dynamics damping="0" friction="0" />
-    </joint>
-    <link name="link_wrist_2">
-        <visual>
-            <origin xyz="0 0 -0.0997" rpy="0 0 0" />
-            <geometry>
-                <mesh filename="file://$(find ros2_robot_ur5e)/meshes/ur5e/visual/wrist2.dae" />
-            </geometry>
-        </visual>
-        <collision>
-            <origin xyz="0 0 -0.0997" rpy="0 0 0" />
-            <geometry>
-                <mesh filename="file://$(find ros2_robot_ur5e)/meshes/ur5e/collision/wrist2.stl" />
-            </geometry>
-        </collision>
-        <inertial>
-            <mass value="1.3" />
-            <origin rpy="0.0 0.0 0.0" xyz="0.0 0.01634 -0.0018" />
-            <inertia
-                ixx="0.0025599" ixy="0.0" ixz="0.0"
-                iyy="0.0025599" iyz="0.0"
-                izz="0.0021942" />
-        </inertial>
-    </link>
-    <joint name="joint_wrist_3" type="revolute">
-        <parent link="link_wrist_2" />
-        <child link="link_wrist_3" />
-        <origin xyz="0 0.09959999999999999 -2.042830148012698e-11" rpy="${pi/2} ${pi} ${pi}" />
-        <axis xyz="0 0 1" />
-        <limit lower="${-2*pi}" upper="${2*pi}" effort="28.0" velocity="${pi}" />
-        <dynamics damping="0" friction="0" />
-    </joint>
-    <link name="link_wrist_3">
-        <visual>
-            <origin xyz="0 0 -0.0989" rpy="${pi/2} 0 0" />
-            <geometry>
-                <mesh filename="file://$(find ros2_robot_ur5e)/meshes/ur5e/visual/wrist3.dae" />
-            </geometry>
-        </visual>
-        <collision>
-            <origin xyz="0 0 -0.0989" rpy="${pi/2} 0 0" />
-            <geometry>
-                <mesh filename="file://$(find ros2_robot_ur5e)/meshes/ur5e/collision/wrist3.stl" />
-            </geometry>
-        </collision>
-        <inertial>
-            <mass value="0.365" />
-            <origin rpy="0.0 0.0 0.0" xyz="0.0 0.0 -0.001159" />
-            <inertia
-                ixx="9.8904140083e-5" ixy="0.0" ixz="0.0"
-                iyy="9.8904140083e-5" iyz="0.0"
-                izz="0.0001321171875" />
-        </inertial>
-    </link>
-    <joint name="joint_ft_frame" type="fixed">
-        <parent link="link_wrist_3" />
-        <child link="link_ft_frame" />
-        <origin xyz="0 0 0" rpy="${pi} 0 0" />
-    </joint>
-    <link name="link_ft_frame" />
-    <joint name="joint_flange" type="fixed">
-        <parent link="link_wrist_3" />
-        <child link="link_flange" />
-        <origin xyz="0 0 0" rpy="0 ${-pi/2} ${-pi/2}" />
-    </joint>
-    <link name="link_flange" />
-    <joint name="joint_tool0" type="fixed">
-        <parent link="link_flange" />
-        <origin xyz="0 0 0" rpy="${pi/2} 0 ${pi/2}" />
-        <child link="link_tool0" />
-    </joint>
-    <link name="link_tool0" />
+    <xacro:arg name="joint_limit_file" default="$(find ros2_robot_ur5e)/config/joint_limits.yaml"/>
+    <xacro:arg name="initial_positions_file" default="$(find ros2_robot_ur5e)/config/initial_positions.yaml"/>
+    <xacro:arg name="ur_calibration_file" default="$(find ros2_robot_ur5e)/config/ur_calibration.yaml"/>
+    <xacro:include filename="robot.ur5e.xacro"/>
+    <xacro:urdf_args
+        joint_limit_file="$(arg joint_limit_file)"
+        ur_calibration_file="$(arg ur_calibration_file)" />
+    <xacro:include filename="robot.control.xacro"/>
+    <xacro:control_args
+        initial_positions_file="$(arg initial_positions_file)" />
 </robot>

Commit message: - add moveit motion planning (movegroup) - add 'tf_prefix', 'namespace' in URDF - add rviz2 launch file

File: description/robot.urdf.xacro (robot description, xacro)
@@ -2,13 +2,22 @@
 <robot xmlns:xacro="http://www.ros.org/wiki/xacro" name="ur5e">
     <link name="world" />
-    <xacro:arg name="joint_limit_file" default="$(find ros2_robot_ur5e)/config/joint_limits.yaml"/>
-    <xacro:arg name="initial_positions_file" default="$(find ros2_robot_ur5e)/config/initial_positions.yaml"/>
-    <xacro:arg name="ur_calibration_file" default="$(find ros2_robot_ur5e)/config/ur_calibration.yaml"/>
-    <xacro:include filename="robot.ur5e.xacro"/>
+    <xacro:arg name="namespace" default="" />
+    <xacro:arg name="tf_prefix" default="" />
+    <xacro:arg name="joint_limit_file" default="$(find ros2_robot_ur5e)/config/joint_limits.yaml" />
+    <xacro:arg name="initial_positions_file" default="$(find ros2_robot_ur5e)/config/initial_positions.yaml" />
+    <xacro:arg name="ur_calibration_file" default="$(find ros2_robot_ur5e)/config/ur_calibration.yaml" />
+    <xacro:include filename="ur5e.urdf.xacro" />
     <xacro:urdf_args
+        tf_prefix="$(arg tf_prefix)"
+        base_xyz="0 0 0"
+        base_rpy="0 0 0"
         joint_limit_file="$(arg joint_limit_file)"
         ur_calibration_file="$(arg ur_calibration_file)" />
-    <xacro:include filename="robot.control.xacro"/>
+    <xacro:include filename="ur5e.control.xacro" />
     <xacro:control_args
+        tf_prefix="$(arg tf_prefix)"
         initial_positions_file="$(arg initial_positions_file)" />
+    <xacro:include filename="gazebo.xacro" />
+    <xacro:gz_args
+        namespace="$(arg namespace)" />
 </robot>

File: description/ur5e.urdf.xacro (robot description, xacro)
@@ -1,5 +1,6 @@
 <?xml version="1.0"?>
 <robot xmlns:xacro="http://www.ros.org/wiki/xacro">
-    <xacro:macro name="urdf_args" params="joint_limit_file ur_calibration_file">
+    <xacro:macro name="urdf_args" params="
+        tf_prefix base_xyz base_rpy joint_limit_file ur_calibration_file">
         <xacro:property name="joint_limits" value="${xacro.load_yaml(joint_limit_file)}"/>
         <xacro:property name="limit_shoulder" value="${joint_limits['joint_limits']['joint_shoulder_pan']}"/>
@@ -16,10 +17,10 @@
         <xacro:property name="origin_wrist_2" value="${calibration['kinematics']['wrist_2']}"/>
         <xacro:property name="origin_wrist_3" value="${calibration['kinematics']['wrist_3']}"/>
-        <joint name="joint_base" type="fixed">
+        <joint name="${tf_prefix}joint_base" type="fixed">
             <parent link="world" />
-            <child link="link_base" />
-            <origin xyz="0 0 0" rpy="0 0 0" />
-        </joint>
-        <link name="link_base">
+            <child link="${tf_prefix}link_base" />
+            <origin xyz="${base_xyz}" rpy="${base_rpy}" />
+        </joint>
+        <link name="${tf_prefix}link_base">
             <visual>
                 <origin xyz="0 0 0" rpy="0 0 ${pi}" />
@@ -43,7 +44,7 @@
             </inertial>
         </link>
-        <joint name="joint_shoulder_pan" type="revolute">
-            <parent link="link_base" />
-            <child link="link_shoulder" />
+        <joint name="${tf_prefix}joint_shoulder_pan" type="revolute">
+            <parent link="${tf_prefix}link_base" />
+            <child link="${tf_prefix}link_shoulder" />
             <origin xyz="${origin_shoulder['x']} ${origin_shoulder['y']} ${origin_shoulder['z']}"
                     rpy="${origin_shoulder['roll']} ${origin_shoulder['pitch']} ${origin_shoulder['yaw']}" />
@@ -53,5 +54,5 @@
             <dynamics damping="0" friction="0" />
         </joint>
-        <link name="link_shoulder">
+        <link name="${tf_prefix}link_shoulder">
             <visual>
                 <origin xyz="0 0 0" rpy="0 0 ${pi}" />
@@ -75,7 +76,7 @@
             </inertial>
         </link>
-        <joint name="joint_shoulder_lift" type="revolute">
-            <parent link="link_shoulder" />
-            <child link="link_upper_arm" />
+        <joint name="${tf_prefix}joint_shoulder_lift" type="revolute">
+            <parent link="${tf_prefix}link_shoulder" />
+            <child link="${tf_prefix}link_upper_arm" />
             <origin xyz="${origin_upper_arm['x']} ${origin_upper_arm['y']} ${origin_upper_arm['z']}"
                     rpy="${origin_upper_arm['roll']} ${origin_upper_arm['pitch']} ${origin_upper_arm['yaw']}" />
@@ -85,5 +86,5 @@
             <dynamics damping="0" friction="0" />
         </joint>
-        <link name="link_upper_arm">
+        <link name="${tf_prefix}link_upper_arm">
             <visual>
                 <origin xyz="0 0 0.138" rpy="${pi/2} 0 ${-pi/2}" />
@@ -107,7 +108,7 @@
             </inertial>
         </link>
-        <joint name="joint_elbow" type="revolute">
-            <parent link="link_upper_arm" />
-            <child link="link_forearm" />
+        <joint name="${tf_prefix}joint_elbow" type="revolute">
+            <parent link="${tf_prefix}link_upper_arm" />
+            <child link="${tf_prefix}link_forearm" />
             <origin xyz="${origin_forearm['x']} ${origin_forearm['y']} ${origin_forearm['z']}"
                     rpy="${origin_forearm['roll']} ${origin_forearm['pitch']} ${origin_forearm['yaw']}" />
@@ -117,5 +118,5 @@
             <dynamics damping="0" friction="0" />
         </joint>
-        <link name="link_forearm">
+        <link name="${tf_prefix}link_forearm">
             <visual>
                 <origin xyz="0 0 0.007" rpy="${pi/2} 0 ${-pi/2}" />
@@ -139,7 +140,7 @@
             </inertial>
         </link>
-        <joint name="joint_wrist_1" type="revolute">
-            <parent link="link_forearm" />
-            <child link="link_wrist_1" />
+        <joint name="${tf_prefix}joint_wrist_1" type="revolute">
+            <parent link="${tf_prefix}link_forearm" />
+            <child link="${tf_prefix}link_wrist_1" />
             <origin xyz="${origin_wrist_1['x']} ${origin_wrist_1['y']} ${origin_wrist_1['z']}"
                     rpy="${origin_wrist_1['roll']} ${origin_wrist_1['pitch']} ${origin_wrist_1['yaw']}" />
@@ -149,5 +150,5 @@
             <dynamics damping="0" friction="0" />
         </joint>
-        <link name="link_wrist_1">
+        <link name="${tf_prefix}link_wrist_1">
             <visual>
                 <origin xyz="0 0 -0.127" rpy="${pi/2} 0 0" />
@@ -171,7 +172,7 @@
             </inertial>
         </link>
-        <joint name="joint_wrist_2" type="revolute">
-            <parent link="link_wrist_1" />
-            <child link="link_wrist_2" />
+        <joint name="${tf_prefix}joint_wrist_2" type="revolute">
+            <parent link="${tf_prefix}link_wrist_1" />
+            <child link="${tf_prefix}link_wrist_2" />
             <origin xyz="${origin_wrist_2['x']} ${origin_wrist_2['y']} ${origin_wrist_2['z']}"
                     rpy="${origin_wrist_2['roll']} ${origin_wrist_2['pitch']} ${origin_wrist_2['yaw']}" />
@@ -181,5 +182,5 @@
             <dynamics damping="0" friction="0" />
         </joint>
-        <link name="link_wrist_2">
+        <link name="${tf_prefix}link_wrist_2">
             <visual>
                 <origin xyz="0 0 -0.0997" rpy="0 0 0" />
@@ -203,7 +204,7 @@
             </inertial>
         </link>
-        <joint name="joint_wrist_3" type="revolute">
-            <parent link="link_wrist_2" />
-            <child link="link_wrist_3" />
+        <joint name="${tf_prefix}joint_wrist_3" type="revolute">
+            <parent link="${tf_prefix}link_wrist_2" />
+            <child link="${tf_prefix}link_wrist_3" />
             <origin xyz="${origin_wrist_3['x']} ${origin_wrist_3['y']} ${origin_wrist_3['z']}"
                     rpy="${origin_wrist_3['roll']} ${origin_wrist_3['pitch']} ${origin_wrist_3['yaw']}" />
@@ -213,5 +214,5 @@
             <dynamics damping="0" friction="0" />
         </joint>
-        <link name="link_wrist_3">
+        <link name="${tf_prefix}link_wrist_3">
             <visual>
                 <origin xyz="0 0 -0.0989" rpy="${pi/2} 0 0" />
@@ -235,22 +236,22 @@
             </inertial>
         </link>
-        <joint name="joint_ft_frame" type="fixed">
-            <parent link="link_wrist_3" />
-            <child link="link_ft_frame" />
+        <joint name="${tf_prefix}joint_ft_frame" type="fixed">
+            <parent link="${tf_prefix}link_wrist_3" />
+            <child link="${tf_prefix}link_ft_frame" />
             <origin xyz="0 0 0" rpy="${pi} 0 0" />
         </joint>
-        <link name="link_ft_frame" />
-        <joint name="joint_flange" type="fixed">
-            <parent link="link_wrist_3" />
-            <child link="link_flange" />
+        <link name="${tf_prefix}link_ft_frame" />
+        <joint name="${tf_prefix}joint_flange" type="fixed">
+            <parent link="${tf_prefix}link_wrist_3" />
+            <child link="${tf_prefix}link_flange" />
             <origin xyz="0 0 0" rpy="0 ${-pi/2} ${-pi/2}" />
         </joint>
-        <link name="link_flange" />
-        <joint name="joint_tool0" type="fixed">
-            <parent link="link_flange" />
+        <link name="${tf_prefix}link_flange" />
+        <joint name="${tf_prefix}joint_tool0" type="fixed">
+            <parent link="${tf_prefix}link_flange" />
             <origin xyz="0 0 0" rpy="${pi/2} 0 ${pi/2}" />
-            <child link="link_tool0" />
-        </joint>
-        <link name="link_tool0" />
+            <child link="${tf_prefix}link_tool0" />
+        </joint>
+        <link name="${tf_prefix}link_tool0" />
     </xacro:macro>
 </robot>
